Commit message: Add debug visuals for mechanical arm

File: sim/mechanical_arm_1_description/urdf/mechanical_arm_1_visual.urdf (robot description, URDF)
Before this commit: robot mechanical_arm_1, 5 links, 4 joints
Links:
- link Link1: geometry collision mesh filename=package://mechanical_arm_1_description/meshes/Link1.STL; visual box size=0.07 0.07 0.075
- link Link2: geometry collision mesh filename=package://mechanical_arm_1_description/meshes/Link2.STL; visual box size=0.09 0.10 0.22
- link Link3: geometry collision mesh filename=package://mechanical_arm_1_description/meshes/Link3.STL; visual box size=0.095 0.095 0.085
- link Link4: geometry collision mesh filename=package://mechanical_arm_1_description/meshes/Link4.STL; visual box size=0.13 0.18 0.16
- link base_link: geometry collision mesh filename=package://mechanical_arm_1_description/meshes/base_link.STL; visual box size=0.065 0.13 0.085

Commit message: Align mechanical arm base axis to Z up

File: sim/mechanical_arm_1_description/urdf/mechanical_arm_1_visual.urdf (robot description, URDF)
Before this commit: robot mechanical_arm_1, 5 links, 4 joints
Links:
- added link arm_base_link, mass 0.054017; collision mesh filename=package://mechanical_arm_1_description/meshes/base_link.STL; visual box size=0.065 0.13 0.085
- link base_link: mass 0.054017 -> None; geometry 
Joints:
- added joint base_axis_fix: type fixed, parent base_link, child arm_base_link, origin xyz=0 0 0 rpy=0 -1.5708 0
- joint j1: parent base_link -> arm_base_link

Commit message: Disable mechanical arm collision geometry

File: sim/mechanical_arm_1_description/urdf/mechanical_arm_1_visual.urdf (robot description, URDF)
Before this commit: robot mechanical_arm_1, 6 links, 5 joints
Links:
- link Link1: geometry visual box size=0.07 0.07 0.075; visual mesh filename=package://mechanical_arm_1_description/meshes/Link1.STL
- link Link2: geometry visual box size=0.09 0.10 0.22; visual mesh filename=package://mechanical_arm_1_description/meshes/Link2.STL
- link Link3: geometry visual box size=0.095 0.095 0.085; visual mesh filename=package://mechanical_arm_1_description/meshes/Link3.STL
- link Link4: geometry visual box size=0.13 0.18 0.16; visual mesh filename=package://mechanical_arm_1_description/meshes/Link4.STL
- link arm_base_link: geometry visual box size=0.065 0.13 0.085; visual mesh filename=package://mechanical_arm_1_description/meshes/base_link.STL

Commit message: Add MoveIt TCP reach validation

File: sim/mechanical_arm_1_description/urdf/mechanical_arm_1_visual.urdf (robot description, URDF)
Before this commit: robot mechanical_arm_1, 6 links, 5 joints
Links:
- added link link4_tip_link
- link Link1: geometry visual mesh filename=package://mechanical_arm_1_description/meshes/Link1.STL
- link Link2: geometry visual mesh filename=package://mechanical_arm_1_description/meshes/Link2.STL
- link Link3: geometry visual mesh filename=package://mechanical_arm_1_description/meshes/Link3.STL
- link Link4: geometry visual mesh filename=package://mechanical_arm_1_description/meshes/Link4.STL
- link arm_base_link: geometry visual mesh filename=package://mechanical_arm_1_description/meshes/base_link.STL
Joints:
- added joint link4_tip_joint: type fixed, parent Link4, child link4_tip_link, origin xyz=-0.100 0.118 0.105 rpy=0 0 0
- joint j2: limit lower=-1.2217 upper=1.2217 effort=2.0 velocity=1.0 -> lower=-1.5708 upper=1.2217 effort=2.0 velocity=1.0
- joint j3: limit lower=-1.2217 upper=1.2217 effort=2.0 velocity=1.0 -> lower=-1.2217 upper=2.6180 effort=2.0 velocity=1.0
